Commit message: materials working

File: src/m2wr_description/urdf/m2wr.xacro (robot description, xacro)
@@ -1,29 +1,5 @@
 <?xml version="1.0" ?>
-<robot name="m2wr"
-    xmlns:xacro="http://www.ros.org/wiki/xacro">
-    <material name="black">
-        <color rgba="0.0 0.0 0.0 1.0"/>
-    </material>
-    <material name="blue">
-        <color rgba="0.203125 0.23828125 0.28515625 1.0"/>
-    </material>
-    <material name="green">
-        <color rgba="0.0 0.8 0.0 1.0"/>
-    </material>
-    <material name="grey">
-        <color rgba="0.2 0.2 0.2 1.0"/>
-    </material>
-    <material name="orange">
-        <color rgba="1.0 0.423529411765 0.0392156862745 1.0"/>
-    </material>
-    <material name="brown">
-        <color rgba="0.870588235294 0.811764705882 0.764705882353 1.0"/>
-    </material>
-    <material name="red">
-        <color rgba="0.80078125 0.12890625 0.1328125 1.0"/>
-    </material>
-    <material name="white">
-        <color rgba="1.0 1.0 1.0 1.0"/>
-    </material>
+<robot name="m2wr" xmlns:xacro="https://www.ros.org/wiki/xacro">
+    <xacro:include filename="$(find m2wr_description)/urdf/materials.xacro"/>
     <gazebo reference="link_chassis">
         <material>Gazebo/Orange</material>

Commit message: macros working

File: src/m2wr_description/urdf/m2wr.xacro (robot description, xacro)
@@ -1,30 +1,8 @@
 <?xml version="1.0" ?>
-<robot name="m2wr" xmlns:xacro="https://www.ros.org/wiki/xacro">
+<robot name="m2wr"
+    xmlns:xacro="https://www.ros.org/wiki/xacro">
     <xacro:include filename="$(find m2wr_description)/urdf/materials.xacro"/>
-    <gazebo reference="link_chassis">
-        <material>Gazebo/Orange</material>
-    </gazebo>
-    <gazebo reference="link_left_wheel">
-        <material>Gazebo/Blue</material>
-    </gazebo>
-    <gazebo reference="link_right_wheel">
-        <material>Gazebo/Blue</material>
-    </gazebo>
-    <gazebo>
-        <plugin filename="libgazebo_ros_diff_drive.so" name="differential_drive_controller">
-            <legacyMode>false</legacyMode>
-            <alwaysOn>true</alwaysOn>
-            <updateRate>20</updateRate>
-            <leftJoint>joint_left_wheel</leftJoint>
-            <rightJoint>joint_right_wheel</rightJoint>
-            <wheelSeparation>0.2</wheelSeparation>
-            <wheelDiameter>0.2</wheelDiameter>
-            <torque>0.1</torque>
-            <commandTopic>cmd_vel</commandTopic>
-            <odometryTopic>odom</odometryTopic>
-            <odometryFrame>odom</odometryFrame>
-            <robotBaseFrame>link_chassis</robotBaseFrame>
-        </plugin>
-    </gazebo>
+    <xacro:include filename="$(find m2wr_description)/urdf/m2wr.gazebo"/>
+    <xacro:include filename="$(find m2wr_description)/urdf/macros.xacro"/>
     <link name="link_chassis">
         <!-- pose and inertial -->
@@ -72,23 +50,5 @@
         </visual>
     </link>
-    <link name="link_right_wheel">
-        <inertial>
-            <mass value="0.2"/>
-            <origin rpy="0 1.5707 1.5707" xyz="0 0 0"/>
-            <inertia ixx="0.000526666666667" ixy="0" ixz="0" iyy="0.000526666666667" iyz="0" izz="0.001"/>
-        </inertial>
-        <collision name="link_right_wheel_collision">
-            <origin rpy="0 1.5707 1.5707" xyz="0 0 0"/>
-            <geometry>
-                <cylinder length="0.04" radius="0.1"/>
-            </geometry>
-        </collision>
-        <visual name="link_right_wheel_visual">
-            <origin rpy="0 1.5707 1.5707" xyz="0 0 0"/>
-            <geometry>
-                <cylinder length="0.04" radius="0.1"/>
-            </geometry>
-        </visual>
-    </link>
+    <xacro:link_wheel name="link_right_wheel"/>
     <joint name="joint_right_wheel" type="continuous">
         <origin rpy="0 0 0" xyz="-0.05 0.15 0"/>
@@ -99,23 +59,5 @@
         <joint_properties damping="1.0" friction="1.0"/>
     </joint>
-    <link name="link_left_wheel">
-        <inertial>
-            <mass value="0.2"/>
-            <origin rpy="0 1.5707 1.5707" xyz="0 0 0"/>
-            <inertia ixx="0.000526666666667" ixy="0" ixz="0" iyy="0.000526666666667" iyz="0" izz="0.001"/>
-        </inertial>
-        <collision name="link_left_wheel_collision">
-            <origin rpy="0 1.5707 1.5707" xyz="0 0 0"/>
-            <geometry>
-                <cylinder length="0.04" radius="0.1"/>
-            </geometry>
-        </collision>
-        <visual name="link_left_wheel_visual">
-            <origin rpy="0 1.5707 1.5707" xyz="0 0 0"/>
-            <geometry>
-                <cylinder length="0.04" radius="0.1"/>
-            </geometry>
-        </visual>
-    </link>
+    <xacro:link_wheel name="link_left_wheel"/>
     <joint name="joint_left_wheel" type="continuous">
         <origin rpy="0 0 0" xyz="-0.05 -0.15 0"/>

Commit message: link_wheel and joint_wheel both working

File: src/m2wr_description/urdf/m2wr.xacro (robot description, xacro)
@@ -51,20 +51,6 @@
     </link>
     <xacro:link_wheel name="link_right_wheel"/>
-    <joint name="joint_right_wheel" type="continuous">
-        <origin rpy="0 0 0" xyz="-0.05 0.15 0"/>
-        <child link="link_right_wheel"/>
-        <parent link="link_chassis"/>
-        <axis rpy="0 0 0" xyz="0 1 0"/>
-        <limit effort="10000" velocity="1000"/>
-        <joint_properties damping="1.0" friction="1.0"/>
-    </joint>
+    <xacro:joint_wheel name="joint_right_wheel" child="link_right_wheel" origin_xyz="-0.05 0.15 0"/>
     <xacro:link_wheel name="link_left_wheel"/>
-    <joint name="joint_left_wheel" type="continuous">
-        <origin rpy="0 0 0" xyz="-0.05 -0.15 0"/>
-        <child link="link_left_wheel"/>
-        <parent link="link_chassis"/>
-        <axis rpy="0 0 0" xyz="0 1 0"/>
-        <limit effort="10000" velocity="1000"/>
-        <joint_properties damping="1.0" friction="1.0"/>
-    </joint>
+    <xacro:joint_wheel name="joint_left_wheel" child="link_left_wheel" origin_xyz="-0.05 -0.15 0"/>
 </robot>

File: src/m2wr_description/urdf/macros.xacro (robot description, xacro)
@@ -22,3 +22,13 @@
         </link>
     </macro>
+    <macro name="joint_wheel" params="name child origin_xyz">
+        <joint name="${name}" type="continuous">
+            <origin rpy="0 0 0" xyz="${origin_xyz}"/>
+            <child link="${child}"/>
+            <parent link="link_chassis"/>
+            <axis rpy="0 0 0" xyz="0 1 0"/>
+            <limit effort="10000" velocity="1000"/>
+            <joint_properties damping="1.0" friction="1.0"/>
+        </joint>
+    </macro>
 </robot>

Commit message: added laser scan readings

File: src/m2wr_description/urdf/m2wr.xacro (robot description, xacro)
@@ -50,4 +50,29 @@
         </visual>
     </link>
+    <link name="sensor_laser">
+        <inertial>
+            <origin xyz="0 0 0" rpy="0 0 0" />
+            <mass value="1" />
+            <xacro:cylinder_inertia mass="1" r="0.05" l="0.1" />
+        </inertial>
+        <visual>
+            <origin xyz="0 0 0" rpy="0 0 0" />
+            <geometry>
+                <cylinder radius="0.05" length="0.1"/>
+            </geometry>
+            <material name="white" />
+        </visual>
+        <collision>
+            <origin xyz="0 0 0" rpy="0 0 0"/>
+            <geometry>
+                <cylinder radius="0.05" length="0.1"/>
+            </geometry>
+        </collision>
+    </link>
+    <joint name="joint_sensor_laser" type="fixed">
+        <origin xyz="0.15 0 0.05" rpy="0 0 0"/>
+        <parent link="link_chassis"/>
+        <child link="sensor_laser"/>
+    </joint>
     <xacro:link_wheel name="link_right_wheel"/>
     <xacro:joint_wheel name="joint_right_wheel" child="link_right_wheel" origin_xyz="-0.05 0.15 0"/>

File: src/m2wr_description/urdf/macros.xacro (robot description, xacro)
@@ -32,3 +32,39 @@
         </joint>
     </macro>
+    <macro name="cylinder_inertia" params="mass r l">
+        <inertia ixx ="${mass*(3*r*r+l*l)/12}" ixy = "0" ixz="0"
+                 iyy ="${mass*(3*r*r+l*l)/12}" iyz="0"
+                 izz ="${mass*(3*r*r+l*l)/12}" />
+    </macro>
+    <gazebo reference="sensor_laser">
+        <sensor type="ray" name="head_hokuyo_sensor">
+            <pose>0 0 0 0 0 0</pose>
+            <visualize>false</visualize>
+            <update_rate>20</update_rate>
+            <ray>
+                <scan>
+                    <horizontal>
+                        <samples>720</samples>
+                        <resolution>1</resolution>
+                        <min_angle>-1.570796</min_angle>
+                        <max_angle>1.570796</max_angle>
+                    </horizontal>
+                </scan>
+                <range>
+                    <min>0.10</min>
+                    <max>10.0</max>
+                    <resolution>0.01</resolution>
+                </range>
+                <noise>
+                    <type>gaussian</type>
+                    <mean>0.0</mean>
+                    <stddev>0.01</stddev>
+                </noise>
+            </ray>
+            <plugin name="gazebo_ros_head_hokuyo_controller" filename="libgazebo_ros_laser.so">
+                <topicName>/m2wr/laser/scan</topicName>
+                <frameName>sensor_laser</frameName>
+            </plugin>
+        </sensor>
+    </gazebo>
 </robot>
