Commit message: CHECKPOINT 2: CARTOGRAPHER 2D Done

File: diff_drive_gazebo/src/m2wr_description/urdf/m2wr.xacro (robot description, xacro)
@@ -6,5 +6,5 @@
     <xacro:include filename="$(find m2wr_description)/urdf/macros.xacro"/>
     <!-- CHASSIS -->
-    <link name="link_chassis">
+    <link name="base_link">
         <!-- pose and inertial -->
         <pose>0 0 0.1 0 0 0</pose>
@@ -74,5 +74,5 @@
     <joint name="joint_sensor_laser" type="fixed">
         <origin xyz="0.15 0 0.05" rpy="0 0 0"/>
-        <parent link="link_chassis"/>
+        <parent link="base_link"/>
         <child link="sensor_laser"/>
     </joint>

File: diff_drive_gazebo/src/m2wr_description/urdf/macros.xacro (robot description, xacro)
@@ -28,5 +28,5 @@
             <origin rpy="0 0 0" xyz="${origin_xyz}"/>
             <child link="${child}"/>
-            <parent link="link_chassis"/>
+            <parent link="base_link"/>
             <axis rpy="0 0 0" xyz="0 1 0"/>
             <limit effort="10000" velocity="1000"/>

Commit message: checking the renaming

File: diff_drive_gazebo/src/m2wr_description/urdf/m2wr.xacro (robot description, xacro)
@@ -6,5 +6,5 @@
     <xacro:include filename="$(find m2wr_description)/urdf/macros.xacro"/>
     <!-- CHASSIS -->
-    <link name="base_link">
+    <link name="link_chassis">
         <!-- pose and inertial -->
         <pose>0 0 0.1 0 0 0</pose>
@@ -74,5 +74,5 @@
     <joint name="joint_sensor_laser" type="fixed">
         <origin xyz="0.15 0 0.05" rpy="0 0 0"/>
-        <parent link="base_link"/>
+        <parent link="link_chassis"/>
         <child link="sensor_laser"/>
     </joint>

File: diff_drive_gazebo/src/m2wr_description/urdf/macros.xacro (robot description, xacro)
@@ -28,5 +28,5 @@
             <origin rpy="0 0 0" xyz="${origin_xyz}"/>
             <child link="${child}"/>
-            <parent link="base_link"/>
+            <parent link="link_chassis"/>
             <axis rpy="0 0 0" xyz="0 1 0"/>
             <limit effort="10000" velocity="1000"/>

Commit message: added lazdar lidar but ROS api not working

File: diff_drive_gazebo/src/m2wr_description/urdf/m2wr.xacro (robot description, xacro)
@@ -2,4 +2,5 @@
 <robot name="m2wr"
     xmlns:xacro="https://www.ros.org/wiki/xacro">
+    <xacro:include filename="$(find m2wr_description)/urdf/laz_rot_lidar.xacro"/>
     <xacro:include filename="$(find m2wr_description)/urdf/materials.xacro"/>
     <xacro:include filename="$(find m2wr_description)/urdf/m2wr.gazebo"/>
@@ -82,3 +83,13 @@
     <xacro:link_wheel name="link_left_wheel"/>
     <xacro:joint_wheel name="joint_left_wheel" child="link_left_wheel" origin_xyz="-0.05 -0.15 0"/>
+<!--
+    LazDar Lidar
+    <!-- <xacro:include filename="$(find m2wr_description)/urdf/laz_rot_lidar.xacro"/> -->
+    <joint name="lidarGlue" type="fixed">
+        <parent link="link_chassis"/>
+        <child link="laz_base"/>
+        <!-- <origin xyz="0 0 ${body_height/2}"/> -->
+        <origin xyz="-0.15 0 0.05" rpy="0 0 0"/>
+    </joint>
+ -->
 </robot>

Commit message: minor commenting error

File: diff_drive_gazebo/src/m2wr_description/urdf/m2wr.xacro (robot description, xacro)
@@ -85,11 +85,9 @@
 <!--
     LazDar Lidar
-    <!-- <xacro:include filename="$(find m2wr_description)/urdf/laz_rot_lidar.xacro"/> -->
+    <xacro:include filename="$(find m2wr_description)/urdf/laz_rot_lidar.xacro"/>
     <joint name="lidarGlue" type="fixed">
         <parent link="link_chassis"/>
         <child link="laz_base"/>
-        <!-- <origin xyz="0 0 ${body_height/2}"/> -->
         <origin xyz="-0.15 0 0.05" rpy="0 0 0"/>
-    </joint>
- -->
+    </joint> -->
 </robot>

Commit message: added Dataspeed velodyne hdl32e +  vlp16 puck

File: diff_drive_gazebo/src/m2wr_description/urdf/m2wr.xacro (robot description, xacro)
@@ -83,5 +83,5 @@
     <xacro:link_wheel name="link_left_wheel"/>
     <xacro:joint_wheel name="joint_left_wheel" child="link_left_wheel" origin_xyz="-0.05 -0.15 0"/>
-<!--
+    <!--
     LazDar Lidar
     <xacro:include filename="$(find m2wr_description)/urdf/laz_rot_lidar.xacro"/>
@@ -91,3 +91,29 @@
         <origin xyz="-0.15 0 0.05" rpy="0 0 0"/>
     </joint> -->
+    <!-- Hokuyo Laser -->
+    <link name="hokuyo_link">
+        <collision>
+            <origin xyz="0 0 0" rpy="0 0 0"/>
+            <geometry>
+                <box size="0.1 0.1 0.1"/>
+            </geometry>
+        </collision>
+        <visual>
+            <origin xyz="0 0 0" rpy="0 0 0"/>
+            <geometry>
+                <mesh filename="package://rrbot_description/meshes/hokuyo.dae"/>
+            </geometry>
+        </visual>
+        <inertial>
+            <mass value="1e-5" />
+            <origin xyz="0 0 0" rpy="0 0 0"/>
+            <inertia ixx="1e-6" ixy="0" ixz="0" iyy="1e-6" iyz="0" izz="1e-6" />
+        </inertial>
+    </link>
+    <joint name="hokuyo_joint" type="fixed">
+        <axis xyz="0 1 0" />
+        <origin xyz="0 0 ${height3 - axel_offset/2}" rpy="0 0 0"/>
+        <parent link="link3"/>
+        <child link="hokuyo_link"/>
+    </joint>
 </robot>

Commit message: trying lidars but lots of protobuf issues

File: diff_drive_gazebo/src/m2wr_description/urdf/m2wr.xacro (robot description, xacro)
@@ -92,4 +92,5 @@
     </joint> -->
     <!-- Hokuyo Laser -->
+<!--
     <link name="hokuyo_link">
         <collision>
@@ -116,4 +117,4 @@
         <parent link="link3"/>
         <child link="hokuyo_link"/>
-    </joint>
+    </joint> -->
 </robot>

Commit message: trying a second world launch

File: diff_drive_gazebo/src/m2wr_description/urdf/m2wr.xacro (robot description, xacro)
@@ -92,5 +92,5 @@
     </joint> -->
     <!-- Hokuyo Lidar-->
-<!--
+    <!--
     <link name="hokuyo_link">
         <collision>
@@ -119,5 +119,10 @@
     </joint> -->
     <!-- Veloddyne Lidar -->
-    <!-- includes the plugin as well -->
+    <!-- Joint -->
     <xacro:include filename="$(find velodyne_description)/urdf/VLP-16.urdf.xacro"/>
+    <VLP-16 parent="link_chassis" name="velodyne" topic="/velodyne_points" hz="10" samples="440" gpu="${gpu}">
+        <origin xyz="0 0 0.4" rpy="0 0 0" />
+    </VLP-16>
+    <!-- includes the urdf and the plugin as well -->
+    <xacro:include filename="$(find velodyne_description)/urdf/example.urdf.xacro"/>
 </robot>

Commit message: created 2nd launch file +  highly modified xacro

File: diff_drive_gazebo/src/m2wr_description/urdf/m2wr.xacro (robot description, xacro)
@@ -52,5 +52,10 @@
         </visual>
     </link>
-    <!-- LAER SENSOR -->
+    <!-- WHEELS -->
+    <xacro:link_wheel name="link_right_wheel"/>
+    <xacro:joint_wheel name="joint_right_wheel" child="link_right_wheel" origin_xyz="-0.05 0.15 0"/>
+    <xacro:link_wheel name="link_left_wheel"/>
+    <xacro:joint_wheel name="joint_left_wheel" child="link_left_wheel" origin_xyz="-0.05 -0.15 0"/>
+    <!-- /////////////////////////////////////// Laser Scanner /////////////////////////////////////////////-->
     <link name="sensor_laser">
         <inertial>
@@ -78,12 +83,6 @@
         <child link="sensor_laser"/>
     </joint>
-    <!-- WHEELS -->
-    <xacro:link_wheel name="link_right_wheel"/>
-    <xacro:joint_wheel name="joint_right_wheel" child="link_right_wheel" origin_xyz="-0.05 0.15 0"/>
-    <xacro:link_wheel name="link_left_wheel"/>
-    <xacro:joint_wheel name="joint_left_wheel" child="link_left_wheel" origin_xyz="-0.05 -0.15 0"/>
-    <!--
-    LazDar Lidar
-    <xacro:include filename="$(find m2wr_description)/urdf/laz_rot_lidar.xacro"/>
+    <!-- /////////////////////////////////////// Lazdar Lidar /////////////////////////////////////////////-->
+    <!-- <xacro:include filename="$(find m2wr_description)/urdf/laz_rot_lidar.xacro"/>
     <joint name="lidarGlue" type="fixed">
         <parent link="link_chassis"/>
@@ -91,5 +90,5 @@
         <origin xyz="-0.15 0 0.05" rpy="0 0 0"/>
     </joint> -->
-    <!-- Hokuyo Lidar-->
+    <!-- /////////////////////////////////////// Hokuyo Lidar /////////////////////////////////////////////-->
     <!--
     <link name="hokuyo_link">
@@ -118,11 +117,39 @@
         <child link="hokuyo_link"/>
     </joint> -->
-    <!-- Veloddyne Lidar -->
+    <!-- /////////////////////////////////////// Veloddyne Lidar /////////////////////////////////////////////-->
+    <xacro:property name="VLP_16_base_radius" value="0.05"/>
+    <xacro:property name="VLP_16_base_height" value="0.05"/>
+    <!-- Constructing a fake base_link -->
+    <joint name="footprint" type="fixed">
+        <parent link="link_chassis"/>
+        <child link="laz_base"/>
+        <origin xyz="-0.15 0 0.05" rpy="0 0 0"/>
+    </joint>
+    <link name="base_link">
+        <inertial>
+            <mass value="0.1"/>
+            <!-- <inertia ixx="0.0" ixy="0.0" ixz="0.0" iyy="0.0" iyz="0.0" izz="0.0"/> -->
+            <inertia ixx="${(1/12) * 0.1 ) (3 * VLP_16_base_radius * VLP_16_base_radius) + VLP_16_base_height * VLP_16_base_height}" ixy="0.0" ixz="0.0" iyy="${(1/12) * 0.1 ) (3 * VLP_16_base_radius * VLP_16_base_radius) + VLP_16_base_height * VLP_16_base_height}" iyz="0.0" izz="${(1/12) * 0.1 * (VLP_16_base_radius * VLP_16_base_radius)}"/>
+        </inertial>
+        <visual>
+            <geometry>
+                <cylinder radius="${VLP_16_base_radius}" length="${VLP_16_base_height}"/>
+            </geometry>
+            <!-- <material name="">
+                <color rgba="1.0 0.0 0.0 1.0"/>
+                <texture filename=""/>
+            </material> -->
+        </visual>
+        <collision>
+            <geometry>
+                <cylinder radius="${VLP_16_base_radius}" length="${VLP_16_base_height}"/>
+            </geometry>
+        </collision>
+    </link>
     <!-- Joint -->
+    <!-- includes the urdf and the plugin as well -->
+    <!-- <xacro:include filename="$(find velodyne_description)/urdf/example.urdf.xacro"/>
     <xacro:include filename="$(find velodyne_description)/urdf/VLP-16.urdf.xacro"/>
     <VLP-16 parent="link_chassis" name="velodyne" topic="/velodyne_points" hz="10" samples="440" gpu="${gpu}">
-        <origin xyz="0 0 0.4" rpy="0 0 0" />
-    </VLP-16>
-    <!-- includes the urdf and the plugin as well -->
-    <xacro:include filename="$(find velodyne_description)/urdf/example.urdf.xacro"/>
+        <origin xyz="0 0 0.4" rpy="0 0 0" /> -->
 </robot>

Commit message: created lidar rviz cofigurations

File: diff_drive_gazebo/src/m2wr_description/urdf/m2wr.xacro (robot description, xacro)
@@ -121,7 +121,7 @@
     <xacro:property name="VLP_16_base_height" value="0.05"/>
     <!-- Constructing a fake base_link -->
-    <joint name="footprint" type="fixed">
+    <joint name="chassis_base_link_joint" type="fixed">
         <parent link="link_chassis"/>
-        <child link="laz_base"/>
+        <child link="base_link"/>
         <origin xyz="-0.15 0 0.05" rpy="0 0 0"/>
     </joint>
@@ -130,5 +130,5 @@
             <mass value="0.1"/>
             <!-- <inertia ixx="0.0" ixy="0.0" ixz="0.0" iyy="0.0" iyz="0.0" izz="0.0"/> -->
-            <inertia ixx="${(1/12) * 0.1 ) (3 * VLP_16_base_radius * VLP_16_base_radius) + VLP_16_base_height * VLP_16_base_height}" ixy="0.0" ixz="0.0" iyy="${(1/12) * 0.1 ) (3 * VLP_16_base_radius * VLP_16_base_radius) + VLP_16_base_height * VLP_16_base_height}" iyz="0.0" izz="${(1/12) * 0.1 * (VLP_16_base_radius * VLP_16_base_radius)}"/>
+            <inertia ixx="${(1/12) * 0.1 * (3 * VLP_16_base_radius * VLP_16_base_radius + VLP_16_base_height * VLP_16_base_height)}" ixy="0" ixz="0" iyy="${(1/12) * 0.1 * (3 * VLP_16_base_radius * VLP_16_base_radius + VLP_16_base_height * VLP_16_base_height)}" iyz="0" izz="${(1/2) * 0.1 * VLP_16_base_radius * VLP_16_base_radius}"/>
         </inertial>
         <visual>
@@ -147,9 +147,10 @@
         </collision>
     </link>
-    <!-- Joint -->
-    <!-- includes the urdf and the plugin as well -->
-    <!-- <xacro:include filename="$(find velodyne_description)/urdf/example.urdf.xacro"/>
+    <!-- Be careful with self-modified lidar -->
+    <xacro:arg name="gpu" default="false"/>
+    <xacro:property name="gpu" value="$(arg gpu)" />
     <xacro:include filename="$(find velodyne_description)/urdf/VLP-16.urdf.xacro"/>
-    <VLP-16 parent="link_chassis" name="velodyne" topic="/velodyne_points" hz="10" samples="440" gpu="${gpu}">
-        <origin xyz="0 0 0.4" rpy="0 0 0" /> -->
+    <VLP-16 parent="base_link" name="velodyne" topic="/velodyne_points" hz="10" samples="440" gpu="${gpu}">
+        <origin xyz="0 0 0.4" rpy="0 0 0" />
+    </VLP-16>
 </robot>

Commit message: visually correct implementation

File: diff_drive_gazebo/src/m2wr_description/urdf/m2wr.xacro (robot description, xacro)
@@ -2,8 +2,10 @@
 <robot name="m2wr"
     xmlns:xacro="https://www.ros.org/wiki/xacro">
+    <!-- /////////////////////////////////////// Importing Urdf/Xacro Dependencies for the robot /////////////////////////////////////////////-->
     <!-- <xacro:include filename="$(find m2wr_description)/urdf/lidar_lazrot.xacro"/> -->
     <xacro:include filename="$(find m2wr_description)/urdf/materials.xacro"/>
     <xacro:include filename="$(find m2wr_description)/urdf/m2wr.gazebo"/>
     <xacro:include filename="$(find m2wr_description)/urdf/macros.xacro"/>
+    <!-- /////////////////////////////////////// Main Body /////////////////////////////////////////////-->
     <!-- CHASSIS -->
     <link name="link_chassis">
@@ -119,5 +121,5 @@
     <!-- /////////////////////////////////////// Veloddyne Lidar /////////////////////////////////////////////-->
     <xacro:property name="VLP_16_base_radius" value="0.05"/>
-    <xacro:property name="VLP_16_base_height" value="0.05"/>
+    <xacro:property name="VLP_16_base_height" value="0.5"/>
     <!-- Constructing a fake base_link -->
     <joint name="chassis_base_link_joint" type="fixed">
@@ -133,4 +135,5 @@
         </inertial>
         <visual>
+            <origin xyz="0.0 0.0 0.20" rpy="0.0 0.0 0.0"/>
             <geometry>
                 <cylinder radius="${VLP_16_base_radius}" length="${VLP_16_base_height}"/>
@@ -142,4 +145,5 @@
         </visual>
         <collision>
+            <origin xyz="0.0 0.0 0.20" rpy="0.0 0.0 0.0"/>
             <geometry>
                 <cylinder radius="${VLP_16_base_radius}" length="${VLP_16_base_height}"/>
@@ -154,3 +158,50 @@
         <origin xyz="0 0 0.4" rpy="0 0 0" />
     </VLP-16>
+    <!-- /////////////////////////////////////// Inertial Measurement Unit /////////////////////////////////////////////-->
+    <!-- joint between the link_chassis and the IMU -->
+    <joint name="link_chassis_IMU_joint" type="fixed">
+        <parent link="link_chassis"/>
+        <child link="imu_sensor"/>
+        <origin xyz="0.0 0.0 0.05" rpy="0.0 0.0 0.0"/>
+        <!-- <axis xyz="0.0 0.0 0.0"/>
+        <limit lower="0.0" upper="0.0" effort="0.0" velocity="0.0"/> -->
+    </joint>
+    <!-- IMU Sensor Link -->
+    <xacro:property name="imu_height" value="0.05"/>
+    <xacro:property name="imu_width" value="0.05"/>
+    <link name="imu_sensor">
+        <inertial>
+            <origin xyz="0.0 0.0 1" rpy="0.0 0.0 0.0"/>
+            <mass value="1.0"/>
+            <inertia ixx="1.0" ixy="0.0" ixz="0.0" iyy="1.0" iyz="0.0" izz="1.0"/>
+        </inertial>
+        <visual>
+            <!-- <origin xyz="0.0 0.0 ${imu_height}" rpy="0.0 0.0 0.0"/> -->
+            <origin xyz="0.0 0.0 0.0" rpy="0.0 0.0 0.0"/>
+            <geometry>
+                <box size="${imu_width} ${imu_width} ${imu_height}"/>
+            </geometry>
+            <!-- <material>
+                <color rgba="28 152 230 1.0"/>
+                <texture filename=""/>
+            </material> -->
+        </visual>
+        <collision>
+            <origin xyz="0.0 0.0 0.0" rpy="0.0 0.0 0.0"/>
+            <geometry>
+                <box size="${imu_width} ${imu_width} ${imu_height}"/>
+            </geometry>
+        </collision>
+    </link>
+    <!-- ROS Built-in Gazebo IMU Plugin Reference -->
+    <gazebo>
+        <plugin name="imu_plugin" filename="libgazebo_ros_imu.so">
+            <alwaysOn>true</alwaysOn>
+            <bodyName>imu_sensor</bodyName>
+            <topicName>imu_topic</topicName>
+            <serviceName>imu_service</serviceName>
+            <gaussianNoise>0.0</gaussianNoise>
+            <updateRate>20</updateRate>
+        </plugin>
+    </gazebo>
 </robot>

Commit message: add inertia name to chassis + caster wheel inertia

File: diff_drive_gazebo/src/m2wr_description/urdf/m2wr.xacro (robot description, xacro)
@@ -12,5 +12,5 @@
         <!-- pose and inertial -->
         <pose>0 0 0.1 0 0 0</pose>
-        <inertial>
+        <inertial name="chassis_inertial">
             <mass value="5"/>
             <origin rpy="0 0 0" xyz="0 0 0.1"/>
@@ -23,4 +23,6 @@
             </geometry>
         </collision>
+        <!-- Naming the visual defaults to white colour -->
+        <!-- <visual name="chassis_visual"> -->
         <visual>
             <origin rpy="0 0 0" xyz="0 0 0"/>
@@ -31,4 +33,9 @@
         </visual>
         <!-- FRONT CASTER WHEEL -->
+        <inertial name="caster_front_inertial">
+            <origin rpy=" 0 0 0" xyz="0.35 0 -0.05"/>
+            <mass value="10.0"/>
+            <inertia ixx="0.0" ixy="0.0" ixz="0.0" iyy="0.0" iyz="0.0" izz="0.0"/>
+        </inertial>
         <collision name="caster_front_collision">
             <origin rpy=" 0 0 0" xyz="0.35 0 -0.05"/>

Commit message: finally a colored model with height extender

File: diff_drive_gazebo/src/m2wr_description/urdf/m2wr.xacro (robot description, xacro)
@@ -30,5 +30,4 @@
                 <box size="0.5 0.3 0.07"/>
             </geometry>
-            <material name="blue"/>
         </visual>
         <!-- FRONT CASTER WHEEL -->
@@ -78,5 +77,4 @@
                 <cylinder radius="0.05" length="0.1"/>
             </geometry>
-            <material name="white" />
         </visual>
         <collision>
